File: Winglet-ESP-HW.kicad_sch (KiCad schematic)
At the start: 4 parts

Commit message: Overhaul for buck-boost converter
Other:
- company: (none) -> TL Embedded
- title: (none) -> Winglet-ESP
Changed lines of the file:
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@@
 	(generator_version "9.0")
 	(paper "A4")
+	(title_block
+		(title "Winglet-ESP")
+		(date "2025-06-03")
+		(rev "v1.0")
+		(company "TL Embedded")
+	)
 	(wire
 		(pts
