File: connector.kicad_sch (KiCad schematic)
At the start: 5 parts, among them M1 Mount_M2.5, M2 Mount_M2.5, U1 24AA01T-I/OT

Commit message: Overhaul for buck-boost converter
Parts:
- removed M1, M2: Mount_M2.5, M_Mechanical:Mount_M2.5, symbol M_Mechanical:Mount_M2.5
- added M1, M2: PTH_M2.5, M_Mechanical:PTH_M2.5, symbol M_Mechanical:PTH_M2.5
Connections:
- net GND: now also M1.1, M2.1
Other:
- company: (none) -> TL Embedded
- title: (none) -> Winglet-ESP
Changed lines of the file:
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@@
 	(generator_version "9.0")
 	(paper "A4")
+	(title_block
+		(title "Winglet-ESP")
+		(rev "v1.0")
+		(company "TL Embedded")
+	)
 	(text_box "+VDDIO: 1.7 - 3.6V\n+BATT: 2.8 - 4.2V\n\nThey may both be 3.3V"
 		(exclude_from_sim no)
@@
 			)
 			(justify left)
+		)
+	)
+	(symbol
+		(lib_id "M_Mechanical:PTH_M2.5")
+		(at 139.7 63.5 270)
+		(unit 1)
+		(exclude_from_sim no)
+		(in_bom no)
+		(on_board yes)
+		(dnp no)
+		(fields_autoplaced yes)
+		(property "Reference" "M2"
+			(at 142.24 62.2299 90)
+			(effects
+				(font
+					(size 1.27 1.27)
+				)
+				(justify left)
+			)
+		)
+		(property "Value" "PTH_M2.5"
+			(at 142.24 64.7699 90)
+			(effects
+				(font
+					(size 1.27 1.27)
+				)
+				(justify left)
+			)
+		)
+		(property "Footprint" "M_Mechanical:PTH_M2.5"
+			(at 133.35 63.5 0)
+			(effects
+				(font
+					(size 1.27 1.27)
+				)
+				(hide yes)
+			)
+		)
+		(property "Datasheet" ""
+			(at 134.62 43.18 0)
+			(effects
+				(font
+					(size 1.27 1.27)
+				)
+				(hide yes)
+			)
+		)
+		(property "Description" ""
+			(at 139.7 63.5 0)
+			(effects
+				(font
+					(size 1.27 1.27)
+				)
+				(hide yes)
+			)
+		)
+		(pin "1"
+		)
+		(instances
+			(project "Winglet-ESP-HW"
+				(path "/6dffa6f3-3b22-4369-8b4c-5139254f6267/511d157f-94fc-4033-97ac-d9db895e7292"
+					(reference "M2")
+					(unit 1)
+				)
+			)
 		)
 	)
@@
 		(dnp no)
 		(fields_autoplaced yes)
-		(property "Reference" "#PWR07"
+		(property "Reference" "#PWR09"
 			(at 224.79 116.84 0)
 			(effects
@@
 			(project "Winglet-ESP-HW"
 				(path "/6dffa6f3-3b22-4369-8b4c-5139254f6267/511d157f-94fc-4033-97ac-d9db895e7292"
-					(reference "#PWR07")
+					(reference "#PWR09")
 					(unit 1)
 				)
@@
 		(dnp no)
 		(fields_autoplaced yes)
-		(property "Reference" "#PWR08"
+		(property "Reference" "#PWR010"
 			(at 224.79 138.43 0)
 			(effects
@@
 		(instances
 			(project ""
+				(path "/6dffa6f3-3b22-4369-8b4c-5139254f6267/511d157f-94fc-4033-97ac-d9db895e7292"
+					(reference "#PWR010")
+					(unit 1)
+				)
+			)
+		)
+	)
+	(symbol
+		(lib_id "power:GND")
+		(at 139.7 67.31 0)
+		(unit 1)
+		(exclude_from_sim no)
+		(in_bom yes)
+		(on_board yes)
+		(dnp no)
+		(property "Reference" "#PWR08"
+			(at 139.7 73.66 0)
+			(effects
+				(font
+					(size 1.27 1.27)
+				)
+				(hide yes)
+			)
+		)
+		(property "Value" "GND"
+			(at 139.7 71.12 0)
+			(effects
+				(font
+					(size 1.27 1.27)
+				)
+			)
+		)
+		(property "Footprint" ""
+			(at 139.7 67.31 0)
+			(effects
+				(font
+					(size 1.27 1.27)
+				)
+				(hide yes)
+			)
+		)
+		(property "Datasheet" ""
+			(at 139.7 67.31 0)
+			(effects
+				(font
+					(size 1.27 1.27)
+				)
+				(hide yes)
+			)
+		)
+		(property "Description" "Power symbol creates a global label with name \"GND\" , ground"
+			(at 139.7 67.31 0)
+			(effects
+				(font
+					(size 1.27 1.27)
+				)
+				(hide yes)
+			)
+		)
+		(pin "1"
+		)
+		(instances
+			(project "Winglet-ESP-HW"
 				(path "/6dffa6f3-3b22-4369-8b4c-5139254f6267/511d157f-94fc-4033-97ac-d9db895e7292"
 					(reference "#PWR08")
@@
 	)
 	(symbol
-		(lib_id "M_Mechanical:Mount_M2.5")
-		(at 139.7 63.5 0)
+		(lib_id "power:GND")
+		(at 139.7 54.61 0)
 		(unit 1)
 		(exclude_from_sim no)
-		(in_bom no)
+		(in_bom yes)
 		(on_board yes)
 		(dnp no)
-		(fields_autoplaced yes)
-		(property "Reference" "M1"
-			(at 142.24 62.2299 0)
-			(effects
-				(font
-					(size 1.27 1.27)
-				)
-				(justify left)
-			)
-		)
-		(property "Value" "Mount_M2.5"
-			(at 142.24 64.7699 0)
-			(effects
-				(font
-					(size 1.27 1.27)
-				)
-				(justify left)
-			)
-		)
-		(property "Footprint" "M_Mechanical:Mount_M2.5"
-			(at 139.7 69.85 0)
+		(property "Reference" "#PWR07"
+			(at 139.7 60.96 0)
+			(effects
+				(font
+					(size 1.27 1.27)
+				)
+				(hide yes)
+			)
+		)
+		(property "Value" "GND"
+			(at 139.7 58.42 0)
+			(effects
+				(font
+					(size 1.27 1.27)
+				)
+			)
+		)
+		(property "Footprint" ""
+			(at 139.7 54.61 0)
 			(effects
 				(font
@@
 		)
 		(property "Datasheet" ""
-			(at 119.38 68.58 0)
-			(effects
-				(font
-					(size 1.27 1.27)
-				)
-				(hide yes)
-			)
-		)
-		(property "Description" ""
-			(at 139.7 63.5 0)
-			(effects
-				(font
-					(size 1.27 1.27)
-				)
-				(hide yes)
-			)
+			(at 139.7 54.61 0)
+			(effects
+				(font
+					(size 1.27 1.27)
+				)
+				(hide yes)
+			)
+		)
+		(property "Description" "Power symbol creates a global label with name \"GND\" , ground"
+			(at 139.7 54.61 0)
+			(effects
+				(font
+					(size 1.27 1.27)
+				)
+				(hide yes)
+			)
+		)
+		(pin "1"
 		)
 		(instances
 			(project "Winglet-ESP-HW"
 				(path "/6dffa6f3-3b22-4369-8b4c-5139254f6267/511d157f-94fc-4033-97ac-d9db895e7292"
-					(reference "M1")
+					(reference "#PWR07")
 					(unit 1)
 				)
@@
 	)
 	(symbol
-		(lib_id "M_Mechanical:Mount_M2.5")
-		(at 139.7 69.85 0)
+		(lib_id "M_Mechanical:PTH_M2.5")
+		(at 139.7 50.8 270)
 		(unit 1)
 		(exclude_from_sim no)
@@
 		(dnp no)
 		(fields_autoplaced yes)
-		(property "Reference" "M2"
-			(at 142.24 68.5799 0)
+		(property "Reference" "M1"
+			(at 142.24 49.5299 90)
 			(effects
 				(font
@@
 			)
 		)
-		(property "Value" "Mount_M2.5"
-			(at 142.24 71.1199 0)
+		(property "Value" "PTH_M2.5"
+			(at 142.24 52.0699 90)
 			(effects
 				(font
@@
 			)
 		)
-		(property "Footprint" "M_Mechanical:Mount_M2.5"
-			(at 139.7 76.2 0)
+		(property "Footprint" "M_Mechanical:PTH_M2.5"
+			(at 133.35 50.8 0)
 			(effects
 				(font
@@
 		)
 		(property "Datasheet" ""
-			(at 119.38 74.93 0)
+			(at 134.62 30.48 0)
 			(effects
 				(font
@@
 		)
 		(property "Description" ""
-			(at 139.7 69.85 0)
-			(effects
-				(font
-					(size 1.27 1.27)
-				)
-				(hide yes)
-			)
+			(at 139.7 50.8 0)
+			(effects
+				(font
+					(size 1.27 1.27)
+				)
+				(hide yes)
+			)
+		)
+		(pin "1"
 		)
 		(instances
-			(project "Winglet-ESP-HW"
+			(project ""
 				(path "/6dffa6f3-3b22-4369-8b4c-5139254f6267/511d157f-94fc-4033-97ac-d9db895e7292"
-					(reference "M2")
+					(reference "M1")
 					(unit 1)
 				)
